Commit message: Add kinimatics class, update dm_driver, cleanup README

File: robot_models/yam/yam.urdf (robot description, URDF)
Before this commit: robot yam, 7 links, 6 joints
Links:
- link base_link: mass 0.82254601869018606486 -> 0.822546; geometry collision mesh filename=package://assets/base_link_collision.stl; visual mesh filename=package://assets/base_link_visual.stl
- link link_1: mass 0.12414973995364896042 -> 0.12415; geometry collision mesh filename=package://assets/link_1_collision.stl; visual mesh filename=package://assets/link_1_visual.stl
- link link_2: mass 1.2443423265581592396 -> 1.24434; geometry collision mesh filename=package://assets/link_2_collision.stl; visual mesh filename=package://assets/link_2_visual.stl
- link link_3: mass 1.08369792994949933451 -> 0.853698; geometry collision mesh filename=package://assets/link_3_collision.stl; visual mesh filename=package://assets/link_3_visual.stl
- link link_4: mass 0.46351139486380599219 -> 0.463511; geometry collision mesh filename=package://assets/link_4_collision.stl; visual mesh filename=package://assets/link_4_visual.stl
- link link_5: mass 0.35096222408098393108 -> 0.350962; geometry collision mesh filename=package://assets/link_5_collision.stl; visual mesh filename=package://assets/link_5_visual.stl
- link link_6: mass 0.60366000667460717466 -> 0.60366; geometry collision mesh filename=package://assets/link_6_collision.stl; visual mesh filename=package://assets/link_6_visual.stl
Joints:
- joint joint1: limit lower=-3.0543261909900767392 upper=2.6179938779914944114 effort=1 velocity=20 -> lower=-2.61799 upper=3.05433 effort=10 velocity=10; origin xyz=6.9387880247888215901e-18 1.8528845721187819917e-22 0.073100000000000026068 rpy=3.141592653589793116 -0 0 -> xyz=-3.55271e-18 -1.05495e-18 0.0631 rpy=0 -0 1.5708
- joint joint2: limit lower=0 upper=3.6651914291880922647 effort=1 velocity=20 -> lower=-3.66519 upper=-0 effort=10 velocity=10; origin xyz=0.033899999999999999578 0.020000000000000028172 -0.040899999999999991918 rpy=-1.570796326794896558 -0 -1.570796326794896558 -> xyz=2.5e-05 -0.02 0.0409 rpy=1.5708 -1.98004e-28 1.5708
- joint joint3: limit lower=0 upper=3.6651914291880922647 effort=1 velocity=20 -> lower=0 upper=3.66519 effort=10 velocity=10; origin xyz=0.26399999999999823608 -3.2057689836051395105e-15 3.2612801348363973375e-16 rpy=-3.1415926535897926719 2.5351744854377732965e-17 1.9081958235744665046e-15 -> xyz=0.264 0 6.77626e-21 rpy=-3.14159 1.26218e-29 7.88861e-31
- joint joint4: limit lower=-1.570796326794896558 upper=1.570796326794896558 effort=1 velocity=20 -> lower=-1.5708 upper=1.5708 effort=10 velocity=10; origin xyz=-0.24499999999999899636 -0.060000260903613045205 -4.7739590058881731238e-15 rpy=3.4875998300716604624e-16 5.3759901509511993963e-16 -2.2204460492502980925e-15 -> xyz=-0.245 -0.0600003 -1.9984e-15 rpy=-5.65471e-31 -1.1507e-13 2.94252e-43
- joint joint5: limit lower=-1.570796326794896558 upper=1.570796326794896558 effort=1 velocity=20 -> lower=-1.5708 upper=1.5708 effort=10 velocity=10; origin xyz=-0.073996827966229070106 -0.039500260903617995245 0.033899473841273959629 rpy=1.570796326794896558 1.570796326794896558 0 -> xyz=-0.0739968 -0.0395003 2.44738e-05 rpy=-1.5708 1.5708 0
- joint joint6: limit lower=-2.0943951023931952626 upper=2.0943951023931952626 effort=1 velocity=20 -> lower=-3.141592653589793 upper=3.141592653589793 effort=10 velocity=10; origin xyz=1.2971278324586327582e-15 -0.025000000000053992921 -0.039500000000001977973 rpy=-1.570796326794896558 -3.8163916471489938501e-16 -2.364019346476597899e-30 -> xyz=-4.0742e-16 0.0353 0.0395 rpy=-1.5708 3.81639e-16 4.68582e-15

Commit message: fix joint limit

File: robot_models/yam/yam.urdf (robot description, URDF)
Before this commit: robot yam_v0, 7 links, 6 joints
Joints:
- joint joint2: limit lower=-3.66519 upper=-0 effort=10 velocity=10 -> lower=0 upper=3.14159 effort=10 velocity=10

Commit message: add some customer change

File: robot_models/yam/yam.urdf (robot description, URDF)
Before this commit: robot yam_v0, 7 links, 6 joints
Joints:
- joint joint1: limit lower=-2.61799 upper=3.05433 effort=10 velocity=10 -> lower=-2.61799 upper=3.13 effort=10 velocity=10
- joint joint2: limit lower=0 upper=3.14159 effort=10 velocity=10 -> lower=0 upper=3.65 effort=10 velocity=10
- joint joint3: limit lower=0 upper=3.66519 effort=10 velocity=10 -> lower=0 upper=3.13 effort=10 velocity=10
- joint joint6: limit lower=-3.141592653589793 upper=3.141592653589793 effort=10 velocity=10 -> lower=-2.0944 upper=2.0944 effort=10 velocity=10
