Commit message: [Release v1.2.2]
Mirror of dev/JH_i2rt-main into the public repo (full-tree file copy; git-ignored files excluded).

Highlights since v1.2.1:
- YAM robot models: re-landed URDF + asset upgrade for yam / yam_pro / yam_ultra
  (new yam_pro.urdf and yam_ultra.urdf, unified base/link1-5 STL naming).
- Encoder: ioheart-complete encoder manager rewrite and new CAN firmware flash tool
  (i2rt/utils/can_flash.py); removed legacy i2rt/utils/encoder_utils.py.
- examples/minimum_gello: teaching-handle support, joint-log mode, and arm/sim modes.
- Dependencies: add crcmod-plus; track uv.lock so `uv sync --locked` is reproducible.
- Tooling: uv-lock/uv-sync + pyright pre-commit hooks, ruff 0.15.4 -> 0.15.6 (hook + CI).

Co-Authored-By: Claude Opus 4.8 (1M context) <noreply@anthropic.com>

File: i2rt/robot_models/arm/yam_ultra/yam_ultra.urdf (robot description, URDF)
Before this commit: robot urdf_top_assembly, 10 links, 9 joints
Links:
- removed link base
- added link ultra_base, mass 0.940115; visual mesh filename=package://urdf_top_assembly/meshes/ultra_base.stl scale=1 1 1
- link link2: mass 1.46908 -> 1.63122
Joints:
- joint dof_joint0: child base -> ultra_base; origin xyz=0 0 0 rpy=0 1.5708 1.5708 -> xyz=-4.16334e-17 0 0 rpy=0 1.5708 -3.57884e-17
- joint dof_joint1: origin xyz=-0.068 -6.80012e-16 -5.41234e-16 rpy=8.32667e-17 2.01874e-17 -3.6657e-17 -> xyz=-0.0733 -1.27793e-15 -8.20164e-16 rpy=1.6619e-16 -2.22045e-16 3.93401e-17; parent base -> ultra_base
- joint dof_joint2: limit lower=-3.9968e-14 upper=3.14159 effort=1 velocity=1 -> lower=-3.14159 upper=3.55271e-15 effort=1 velocity=1; origin xyz=-0.0455 -0.0339 -0.02 rpy=4.86604e-16 3.99049e-14 -3.14159 -> xyz=-0.0455 0.03285 -0.02 rpy=-6.12812e-16 1.38778e-16 4.61357e-15
- joint dof_joint3: limit lower=0 upper=3.14159 effort=1 velocity=1 -> lower=0 upper=3.66519 effort=1 velocity=1; origin xyz=4.08431e-07 -0.0688 0.264 rpy=-1.01074e-14 7.11653e-14 -3.14159 -> xyz=4.08431e-07 -0.0678 0.264 rpy=-9.81467e-15 6.80289e-14 -9.61378e-18
- joint dof_joint4: origin xyz=-0.0600003 -0.0688 -0.244999 rpy=1.03997e-14 -8.62366e-14 -4.39823e-15 -> xyz=-0.0600003 0.0678 -0.244999 rpy=4.17957e-15 -6.65093e-14 -6.51788e-15
- joint dof_joint5: axis -1 0 0 -> 1 0 0; origin xyz=-0.0405003 0.0338995 -0.0739989 rpy=-2.58127e-15 -1.37665e-15 -1.04686e-15 -> xyz=-0.0403003 -0.0338507 -0.0703851 rpy=-3.44701e-15 -5.07057e-15 -5.25136e-15
- joint dof_joint6: origin xyz=0.0404996 2.39858e-07 -0.0356 rpy=1.00451e-15 -4.22055e-16 -1.11022e-16 -> xyz=0.0404996 2.39858e-07 -0.0419481 rpy=1.01308e-15 -1.77514e-15 8.61476e-15
- joint dof_joint7: origin xyz=-0.0239931 0.0445119 -0.0566829 rpy=1.08798e-14 2.77556e-15 5.77825e-15 -> xyz=0.0239931 -0.0445119 -0.0566919 rpy=-5.56846e-15 -3.16067e-15 3.14159
- joint dof_joint8: origin xyz=0.0239931 -0.0445119 -0.0566829 rpy=2.05045e-15 1.32394e-14 -3.16199e-14 -> xyz=-0.0239931 0.0445119 -0.0566829 rpy=-9.13119e-15 1.66533e-16 -3.14159

Commit message: fix(yam_ultra): point base link/mesh at existing base.stl asset
- i2rt/robot_models/arm/yam_ultra/yam_ultra.urdf: renamed link `ultra_base` to `base` and mesh `ultra_base.stl` to `base.stl` (including parent/child joint refs) so the URDF references the mesh that actually exists in assets/base.stl instead of a dangling ultra_base.stl

Closes ROB-1546

Co-authored-by: Claude Opus 4.8 <noreply@anthropic.com>

File: i2rt/robot_models/arm/yam_ultra/yam_ultra.urdf (robot description, URDF)
Before this commit: robot urdf_top_assembly, 10 links, 9 joints
Links:
- removed link ultra_base
- added link base, mass 0.940115; visual mesh filename=package://urdf_top_assembly/meshes/base.stl scale=1 1 1
Joints:
- joint dof_joint0: child ultra_base -> base
- joint dof_joint1: parent ultra_base -> base
