Commit message: fix(models): correct YAM joint 2/3/1/4 limits to measured values
Bench testing showed the real joint working ranges differ from what the
model files encoded, and the .xml / .urdf files were also inconsistent
with each other across variants. Unify Standard / Pro / Ultra to the
measured limits:

  joint1:  -150° to  180°   (was upper 175°)
  joint2:     0° to  210°   (was 180° / 209°, inconsistent)
  joint3:     0° to  180°   (was 210°)
  joint4:   -97° to   90°   (was -90°)
  joint5:   -90° to   90°   (unchanged)
  joint6:  -120° to  120°   (unchanged)

Both the MuJoCo .xml (authoritative — the SDK enforces limits from here)
and the .urdf (external viz) are updated. While fixing magnitudes, two
clearly-broken URDF ranges were also corrected to match:
  - yam_pro.urdf  joint3: was [-360°, 210°]  → [0°, 180°]
  - yam_ultra.urdf joint2: was [-180°, 0°] (reversed) → [0°, 210°]

BIG YAM is intentionally left unchanged (different mechanics — DM6248
shoulders, reversed joints — pending its own bench measurement).

Verified: all three models load in MuJoCo and report the expected
compiled joint ranges.

Co-Authored-By: Claude Sonnet 4.6 <noreply@anthropic.com>

File: i2rt/robot_models/arm/yam/yam.urdf (robot description, URDF)
Before this commit: robot urdf_top_assembly, 10 links, 9 joints
Joints:
- joint dof_joint1: limit lower=-2.61799 upper=3.05433 effort=1 velocity=1 -> lower=-2.61799 upper=3.14159 effort=1 velocity=1
- joint dof_joint2: limit lower=-3.9968e-14 upper=3.14159 effort=1 velocity=1 -> lower=0 upper=3.66519 effort=1 velocity=1
- joint dof_joint4: limit lower=-1.5708 upper=1.5708 effort=1 velocity=1 -> lower=-1.69297 upper=1.5708 effort=1 velocity=1

File: i2rt/robot_models/arm/yam_pro/yam_pro.urdf (robot description, URDF)
Before this commit: robot urdf_top_assembly, 21 links, 20 joints
Joints:
- joint dof_joint1: limit lower=-2.61799 upper=3.05433 effort=1 velocity=1 -> lower=-2.61799 upper=3.14159 effort=1 velocity=1
- joint dof_joint2: limit lower=0 upper=3.14159 effort=1 velocity=1 -> lower=0 upper=3.66519 effort=1 velocity=1
- joint dof_joint3: limit lower=-6.28319 upper=3.66519 effort=1 velocity=1 -> lower=0 upper=3.14159 effort=1 velocity=1
- joint dof_joint4: limit lower=-1.5708 upper=1.5708 effort=1 velocity=1 -> lower=-1.69297 upper=1.5708 effort=1 velocity=1

File: i2rt/robot_models/arm/yam_ultra/yam_ultra.urdf (robot description, URDF)
Before this commit: robot urdf_top_assembly, 10 links, 9 joints
Joints:
- joint dof_joint1: limit lower=-2.61799 upper=3.05433 effort=1 velocity=1 -> lower=-2.61799 upper=3.14159 effort=1 velocity=1
- joint dof_joint2: limit lower=-3.14159 upper=3.55271e-15 effort=1 velocity=1 -> lower=0 upper=3.66519 effort=1 velocity=1
- joint dof_joint3: limit lower=0 upper=3.66519 effort=1 velocity=1 -> lower=0 upper=3.14159 effort=1 velocity=1
- joint dof_joint4: limit lower=-1.5708 upper=1.5708 effort=1 velocity=1 -> lower=-1.69297 upper=1.5708 effort=1 velocity=1
