Commit message: [Release v1.2.4]
Mirror of dev/JH_i2rt-main into the public repo. Highlights since v1.2.3:

- YAM family URDF/MJCF frame alignment + ONShape alignment pipeline (#46):
  new align-urdf-mjcf / transform-onshape-urdf skills, per-arm robot_models
  READMEs, URDF↔MJCF alignment tests, regenerated models/assets, project CLAUDE.md.
- minimum_gello: drop stale follower commands to stop growing teleop lag (#47),
  with test_minimum_gello_lag.py.
- Remove stale gripper_collision.stl from crank_4310.

Co-authored-by: Claude Opus 4.8 <noreply@anthropic.com>

File: i2rt/robot_models/arm/big_yam/big_yam.urdf (robot description, URDF)
Before this commit: robot output, 9 links, 8 joints
Joints:
- joint joint1: axis 0 0 1 -> 0 0 -1; limit lower=-2.61799 upper=3.05433 effort=10 velocity=10 -> lower=-2.87979 upper=2.87979 effort=10 velocity=10
- joint joint3: limit lower=0 upper=3.14159 effort=10 velocity=10 -> lower=0 upper=3.01942 effort=10 velocity=10
- joint joint4: axis 0 0 1 -> 0 0 -1; limit lower=-1.5708 upper=1.5708 effort=10 velocity=10 -> lower=-1.69297 upper=1.5708 effort=10 velocity=10
- joint joint5: axis 0 0 1 -> 0 0 -1

File: i2rt/robot_models/arm/yam/yam.urdf (robot description, URDF)
Before this commit: robot urdf_top_assembly, 10 links, 9 joints
Links:
- removed link root
- link base: geometry visual mesh filename=assets/base.stl scale=1 1 1
- link gripper: geometry visual mesh filename=assets/gripper.stl scale=1 1 1
- link link1: geometry visual mesh filename=assets/link1.stl scale=1 1 1
- link link2: geometry visual mesh filename=assets/link2.stl scale=1 1 1
- link link3: geometry visual mesh filename=assets/link3.stl scale=1 1 1
- link link4: geometry visual mesh filename=assets/link4.stl scale=1 1 1
- link link5: geometry visual mesh filename=assets/link5.stl scale=1 1 1
- link tip_left: geometry visual mesh filename=assets/tip_left.stl scale=1 1 1
- link tip_right: geometry visual mesh filename=assets/tip_right.stl scale=1 1 1
Joints:
- removed joint dof_joint0
- removed joint dof_joint1
- removed joint dof_joint2
- removed joint dof_joint3
- removed joint dof_joint4
- removed joint dof_joint5
- removed joint dof_joint6
- removed joint dof_joint7
- removed joint dof_joint8
- added joint joint1: type revolute, parent base, child link1, origin xyz=-2.49777947129965e-07 -9.17402363407408e-13 0.0679999999995413 rpy=0 1.5708 3.1415963267949, axis -1 0 0, limit lower=-2.61799 upper=3.14159 effort=1 velocity=1
- added joint joint2: type revolute, parent link1, child link2, origin xyz=-0.0455 -0.0339 -0.02 rpy=-1.7953e-16 5.55112e-17 -3.14159, axis 3.58252e-15 1 -3.2007e-16, limit lower=-8.88178e-16 upper=3.66519 effort=1 velocity=1
- added joint joint3: type revolute, parent link2, child link3, origin xyz=4.08431e-07 -0.0688 0.264 rpy=-2.99502e-14 -1.6015e-14 -3.14159, axis 4.54273e-15 1 1.04275e-14, limit lower=0 upper=3.14159 effort=1 velocity=1
- added joint joint4: type revolute, parent link3, child link4, origin xyz=-0.0600003 -0.0688 -0.244999 rpy=2.95536e-14 8.52374e-14 -2.10585e-14, axis 0 1 0, limit lower=-1.69297 upper=1.5708 effort=1 velocity=1
- added joint joint5: type revolute, parent link4, child link5, origin xyz=-0.0405003 0.0338995 -0.0739989 rpy=2.73264e-14 -4.32956e-16 -8.32667e-17, axis 1 0 0, limit lower=-1.5708 upper=1.5708 effort=1 velocity=1
- added joint joint6: type revolute, parent link5, child gripper, origin xyz=0.0404996 2.39858e-07 -0.0356 rpy=8.83309e-16 -5.88588e-16 7.69861e-14, axis 1.46014e-15 2.40808e-14 -1, limit lower=-2.0944 upper=2.0944 effort=1 velocity=1
- added joint joint7: type prismatic, parent gripper, child tip_left, origin xyz=-0.0239931 0.0445119 -0.0566829 rpy=1.02229e-14 4.71845e-16 1.68314e-15, axis 6.86541e-15 1 0, limit lower=-0.04695 upper=4.60927e-15 effort=1 velocity=1
- added joint joint8: type prismatic, parent gripper, child tip_right, origin xyz=0.0239931 -0.0445119 -0.0566829 rpy=9.6084e-15 -2.77556e-16 -3.77189e-15, axis -6.86541e-15 -1 0, limit lower=-0.04695 upper=0 effort=1 velocity=1

File: i2rt/robot_models/arm/yam_pro/yam_pro.urdf (robot description, URDF)
Before this commit: robot urdf_top_assembly, 21 links, 20 joints
Links:
- removed link base_1
- removed link gripper_1
- removed link link1_1
- removed link link2_1
- removed link link3_1
- removed link link4_1
- removed link link5_1
- removed link root
- removed link tip_left_1
- removed link tip_left_2
- removed link tip_right_1
- removed link tip_right_2
- link base: geometry visual mesh filename=assets/base.stl scale=1 1 1
- link gripper: geometry visual mesh filename=assets/gripper.stl scale=1 1 1
- link link1: geometry visual mesh filename=assets/link1.stl scale=1 1 1
- link link2: geometry visual mesh filename=assets/link2.stl scale=1 1 1
- link link3: geometry visual mesh filename=assets/link3.stl scale=1 1 1
- link link4: geometry visual mesh filename=assets/link4.stl scale=1 1 1
- link link5: mass 0.395939 -> 0.403307; geometry visual mesh filename=assets/link5.stl scale=1 1 1
- link tip_left: geometry visual mesh filename=assets/tip_left.stl scale=1 1 1
- link tip_right: geometry visual mesh filename=assets/tip_right.stl scale=1 1 1
Joints:
- removed joint dof_joint0
- removed joint dof_joint1
- removed joint dof_joint2
- removed joint dof_joint3
- removed joint dof_joint4
- removed joint dof_joint5
- removed joint dof_joint6
- removed joint dof_joint7
- removed joint dof_joint8
- removed joint 分组_1_fastened_joint
- removed joint 分组_1_fastened_joint_1
- removed joint 分组_1_fastened_joint_2
- removed joint 分组_1_fastened_joint_3
- removed joint 分组_1_fastened_joint_4
- removed joint 分组_1_fastened_joint_5
- removed joint 分组_1_fastened_joint_6
- removed joint 分组_1_fastened_joint_7
- removed joint 分组_1_fastened_joint_8
- removed joint 分组_1_fastened_joint_9
- removed joint 紧固_2
- added joint joint1: type revolute, parent base, child link1, origin xyz=-2.49777947114e-07 0 0.0679999999995 rpy=-3.14159265359 1.57079265359 2.65359006568e-06, axis -1 0 0, limit lower=-2.61799 upper=3.14159 effort=1 velocity=1
- added joint joint2: type revolute, parent link1, child link2, origin xyz=-0.0455 -0.0329 -0.02 rpy=3.36235e-16 -1.91164e-15 3.46073e-15, axis -3.58252e-15 -1 3.35753e-16, limit lower=0 upper=3.66519 effort=1 velocity=1
- added joint joint3: type revolute, parent link2, child link3, origin xyz=4.08431e-07 -0.00205 0.264 rpy=-1.07982e-14 5.71487e-14 6.40141e-16, axis 4.54273e-15 1 1.04275e-14, limit lower=0 upper=3.14159 effort=1 velocity=1
- added joint joint4: type revolute, parent link3, child link4, origin xyz=-0.0600003 0.0688 -0.244999 rpy=1.04275e-14 -3.65263e-14 -4.34003e-15, axis 0 1 0, limit lower=-1.69297 upper=1.5708 effort=1 velocity=1
- added joint joint5: type revolute, parent link4, child link5, origin xyz=-0.0403003 -0.0338507 -0.0739989 rpy=-8.38162e-15 -2.23269e-15 -3.35842e-15, axis 1 0 0, limit lower=-1.5708 upper=1.5708 effort=1 velocity=1
- added joint joint6: type revolute, parent link5, child gripper, origin xyz=0.0404996 2.39858e-07 -0.0356 rpy=6.79401e-15 -1.7587e-15 8.19623e-15, axis 1.46014e-15 2.40808e-14 -1, limit lower=-2.0944 upper=2.0944 effort=1 velocity=1
- added joint joint7: type prismatic, parent gripper, child tip_left, origin xyz=0.0239931 -0.0445119 -0.0566829 rpy=-8.79052e-15 2.82248e-16 3.14159, axis 6.86541e-15 1 0, limit lower=-0.04695 upper=0 effort=1 velocity=1
- added joint joint8: type prismatic, parent gripper, child tip_right, origin xyz=-0.0239931 0.0445119 -0.0566829 rpy=-9.31451e-15 -5.70393e-16 -3.14159, axis -6.86541e-15 -1 0, limit lower=-0.04695 upper=1.58391e-15 effort=1 velocity=1

File: i2rt/robot_models/arm/yam_ultra/yam_ultra.urdf (robot description, URDF)
Before this commit: robot urdf_top_assembly, 10 links, 9 joints
Links:
- removed link root
- link base: geometry visual mesh filename=assets/base.stl scale=1 1 1
- link gripper: geometry visual mesh filename=assets/gripper.stl scale=1 1 1
- link link1: geometry visual mesh filename=assets/link1.stl scale=1 1 1
- link link2: geometry visual mesh filename=assets/link2.stl scale=1 1 1
- link link3: geometry visual mesh filename=assets/link3.stl scale=1 1 1
- link link4: geometry visual mesh filename=assets/link4.stl scale=1 1 1
- link link5: geometry visual mesh filename=assets/link5.stl scale=1 1 1
- link tip_left: geometry visual mesh filename=assets/tip_left.stl scale=1 1 1
- link tip_right: geometry visual mesh filename=assets/tip_right.stl scale=1 1 1
Joints:
- removed joint dof_joint0
- joint dof_joint1: limit lower=-2.61799 upper=3.05433 effort=1 velocity=1 -> lower=-2.61799 upper=3.14159 effort=1 velocity=1; origin xyz=-0.0733 -1.27793e-15 -8.20164e-16 rpy=1.6619e-16 -2.22045e-16 3.93401e-17 -> xyz=0 0 0.0733 rpy=0 1.57079632679 3.14159265359
- joint dof_joint2: axis 3.58252e-15 1 -3.2007e-16 -> -3.58252e-15 -1 3.2007e-16; limit lower=-3.14159 upper=3.55271e-15 effort=1 velocity=1 -> lower=0 upper=3.66519 effort=1 velocity=1; origin xyz=-0.0455 0.03285 -0.02 rpy=-6.12812e-16 1.38778e-16 4.61357e-15 -> xyz=-0.0455 0.03285 -0.02 rpy=-4.21325e-15 -1.5065e-29 9.98062e-15
- joint dof_joint3: limit lower=0 upper=3.66519 effort=1 velocity=1 -> lower=0 upper=3.14159 effort=1 velocity=1; origin xyz=4.08431e-07 -0.0678 0.264 rpy=-9.81467e-15 6.80289e-14 -9.61378e-18 -> xyz=4.08431e-07 -0.0678 0.264 rpy=-6.20015e-15 6.98506e-29 -5.07758e-15
- joint dof_joint4: limit lower=-1.5708 upper=1.5708 effort=1 velocity=1 -> lower=-1.69297 upper=1.5708 effort=1 velocity=1; origin xyz=-0.0600003 0.0678 -0.244999 rpy=4.17957e-15 -6.65093e-14 -6.51788e-15 -> xyz=-0.0600003 0.0678 -0.244999 rpy=1.04275e-14 -2.77556e-17 -4.04405e-15
- joint dof_joint5: origin xyz=-0.0403003 -0.0338507 -0.0703851 rpy=-3.44701e-15 -5.07057e-15 -5.25136e-15 -> xyz=-0.0403003 -0.0338507 -0.0703851 rpy=-1.02186e-14 2.77556e-17 -6.12323e-17
- joint dof_joint6: axis -1.46014e-15 -2.40808e-14 1 -> 1.46014e-15 2.40808e-14 -1; origin xyz=0.0404996 2.39858e-07 -0.0419481 rpy=1.01308e-15 -1.77514e-15 8.61476e-15 -> xyz=0.0404996 2.39858e-07 -0.0419481 rpy=7.6222e-29 -5.3963e-29 4.42535e-15
- joint dof_joint7: limit lower=-0.04695 upper=0 effort=1 velocity=1 -> lower=-0.04695 upper=1.84314e-18 effort=1 velocity=1; origin xyz=0.0239931 -0.0445119 -0.0566919 rpy=-5.56846e-15 -3.16067e-15 3.14159 -> xyz=0.0239931 -0.0445119 -0.0566919 rpy=-9.48894e-15 -1.66533e-16 3.14159
- joint dof_joint8: limit lower=-0.04695 upper=0 effort=1 velocity=1 -> lower=-0.04695 upper=8.78204e-18 effort=1 velocity=1; origin xyz=-0.0239931 0.0445119 -0.0566829 rpy=-9.13119e-15 1.66533e-16 -3.14159 -> xyz=-0.0239931 0.0445119 -0.0566829 rpy=-9.13119e-15 4.4964e-15 -3.14159
