Commit message: [Release v1.3.4]
Mirror of dev/JH_i2rt-main into the public repo.

- i2rt/robot_models/station/assets/: replace the six per-part D405 STLs with three
  pre-baked assembly meshes (d405_top, d405_wrist_crank_4310, d405_wrist_linear_4310),
  each sitting at identity in its camera body
- i2rt/robot_models/station/yam_station_{crank,linear}_4310_d405/: collapse each
  station camera to one mesh and one frame so the optical frame and the geometry
  frame coincide; refresh the extrinsics READMEs
- i2rt/robot_models/gripper/{crank,linear,flexible}_4310/*.xml: drop the d405
  sub-model includes now folded into the station models
- i2rt/robot_models/arm/yam/v1/: remove the superseded per-arm d405 variants

Co-Authored-By: Claude Opus 5 (1M context) <noreply@anthropic.com>

File: i2rt/robot_models/station/yam_station_crank_4310_d405/yam_station_crank_4310_d405.urdf (robot description, URDF)
Before this commit: robot yam_station_crank_4310_d405, 29 links, 28 joints
Links:
- removed link left_camera_body
- removed link left_camera_bracket
- removed link left_camera_cable_holder
- removed link right_camera_body
- removed link right_camera_bracket
- removed link right_camera_cable_holder
- removed link top_camera_body
- removed link top_camera_bracket
- link left_camera: mass 1e-09 -> 6.570123e-05; geometry visual mesh filename=../assets/d405_wrist_crank_4310.stl scale=1 1 1
- link right_camera: mass 1e-09 -> 6.570123e-05; geometry visual mesh filename=../assets/d405_wrist_crank_4310.stl scale=1 1 1
- link top_camera: mass 1e-09 -> 7.36722e-05; geometry visual mesh filename=../assets/d405_top.stl scale=1 1 1
Joints:
- removed joint left_camera_body_joint
- removed joint left_camera_bracket_joint
- removed joint left_camera_cable_holder_joint
- removed joint right_camera_body_joint
- removed joint right_camera_bracket_joint
- removed joint right_camera_cable_holder_joint
- removed joint top_camera_body_joint
- removed joint top_camera_bracket_joint
- joint left_camera_joint: origin xyz=-0.009 0 0 rpy=3.14159 0 0 -> xyz=-0.07972864298920912 0.0016999000000607195 -0.06602077467211452 rpy=2.268922 3.673205103416066e-06 1.5707963267814042; parent left_camera_body -> left_gripper
- joint right_camera_joint: origin xyz=-0.009 0 0 rpy=3.14159 0 0 -> xyz=-0.07972864298920912 0.0016999000000607195 -0.06602077467211452 rpy=2.268922 3.673205103416066e-06 1.5707963267814042; parent right_camera_body -> right_gripper
- joint top_camera_joint: axis 0 0 1 -> (none); origin xyz=0.001 2.22045e-16 -0.022 rpy=3.14159 4.85103e-33 -2.80074e-33 -> xyz=-0.16649488039785276 -0.3050000004052651 0.9543205295851617 rpy=-2.6179963071795864 -2.220446049250313e-16 -1.5708; parent top_camera_body -> left_base

File: i2rt/robot_models/station/yam_station_linear_4310_d405/yam_station_linear_4310_d405.urdf (robot description, URDF)
Before this commit: robot yam_station_linear_4310_d405, 31 links, 30 joints
Links:
- removed link left_camera_body
- removed link left_camera_bracket
- removed link left_camera_cable_holder
- removed link left_camera_cover
- removed link right_camera_body
- removed link right_camera_bracket
- removed link right_camera_cable_holder
- removed link right_camera_cover
- removed link top_camera_body
- removed link top_camera_bracket
- link left_camera: mass 1e-09 -> 6.946694e-05; geometry visual mesh filename=../assets/d405_wrist_linear_4310.stl scale=1 1 1
- link right_camera: mass 1e-09 -> 6.946694e-05; geometry visual mesh filename=../assets/d405_wrist_linear_4310.stl scale=1 1 1
- link top_camera: mass 1e-09 -> 7.36722e-05; geometry visual mesh filename=../assets/d405_top.stl scale=1 1 1
Joints:
- removed joint left_camera_body_joint
- removed joint left_camera_bracket_joint
- removed joint left_camera_cable_holder_joint
- removed joint left_camera_cover_joint
- removed joint right_camera_body_joint
- removed joint right_camera_bracket_joint
- removed joint right_camera_cable_holder_joint
- removed joint right_camera_cover_joint
- removed joint top_camera_body_joint
- removed joint top_camera_bracket_joint
- joint left_camera_joint: axis 0 0 1 -> (none); origin xyz=-0.019 0 -0.023 rpy=3.14159 1.57772e-30 -4.73317e-30 -> xyz=-0.07043497874827391 -7.656797949839866e-08 -0.07700592901799347 rpy=2.70525 3.673205103638111e-06 1.5707963267814136; parent left_camera_body -> left_gripper
- joint right_camera_joint: axis 0 0 1 -> (none); origin xyz=-0.019 0 -0.023 rpy=3.14159 1.57772e-30 -4.73317e-30 -> xyz=-0.07043497874827391 -7.656797949839866e-08 -0.07700592901799347 rpy=2.70525 3.673205103638111e-06 1.5707963267814136; parent right_camera_body -> right_gripper
- joint top_camera_joint: axis 0 0 1 -> (none); origin xyz=0.001 2.22045e-16 -0.022 rpy=3.14159 4.85103e-33 -2.80074e-33 -> xyz=-0.16649488039785276 -0.3050000004052651 0.9543205295851617 rpy=-2.6179963071795864 -2.220446049250313e-16 -1.5708; parent top_camera_body -> left_base
