Commit message: [Release v1.3.6]
Mirror of dev/JH_i2rt-main into the public repo. Carries dev #63: every arm's
flange frame moves to the z-forward tool convention (+X right, +Y down,
+Z forward), and the arm/gripper model literals are simplified to the
exporter's own 6-significant-digit precision.

Nothing moves physically -- the frame turns by R_fix and everything expressed
in it is counter-rotated by the same matrix -- but the orientation a consumer
reads off the terminal `gripper` body differs from v1.3.5.

Co-Authored-By: Claude Opus 5 (1M context) <noreply@anthropic.com>

File: i2rt/robot_models/arm/big_yam/v1/big_yam.urdf (robot description, URDF)
Before this commit: robot output, 9 links, 8 joints
Joints:
- joint joint1: origin xyz=-0 -0 0.0666 rpy=3.14159 -0 0 -> xyz=0 0 0.0666 rpy=3.14159 0 0
- joint joint2: origin xyz=0.0219115 0.022425 -0.0639519 rpy=1.5708 0 -0 -> xyz=0.0219115 0.022425 -0.0639519 rpy=1.5708 0 0
- joint joint5: origin xyz=0.0739989 -0.0403003 0.0323887 rpy=1.5708 -0 0 -> xyz=0.0739989 -0.0403003 0.0323887 rpy=1.5708 0 0
- joint joint6: origin xyz=0.0356 -2.39858e-07 -0.0404996 rpy=-1.5708 0 1.5708 -> xyz=0.0356 0 -0.0404996 rpy=-1.5708 0 -1.5708
- joint joint7: origin xyz=-0.0239931 0.0450619 -0.0566829 rpy=-1.5708 1.5708 0 -> xyz=0.0239931 0.0450619 0.0566829 rpy=-1.5708 -1.5708 0
- joint joint8: origin xyz=0.0239931 -0.0450619 -0.0566829 rpy=1.5708 1.5708 0 -> xyz=-0.0239931 -0.0450619 0.0566829 rpy=1.5708 -1.5708 0

File: i2rt/robot_models/arm/yam/v1/yam.urdf (robot description, URDF)
Before this commit: robot yam, 9 links, 8 joints
Joints:
- joint joint1: origin xyz=-2.49777947129965e-07 -9.17402363407408e-13 0.0679999999995413 rpy=0 1.5708 3.1415963267949 -> xyz=0 0 0.068 rpy=0 1.5708 3.1416
- joint joint2: axis 3.58252e-15 1 -3.2007e-16 -> 0 1 0; origin xyz=-0.0455 -0.0339 -0.02 rpy=-1.7953e-16 5.55112e-17 -3.14159 -> xyz=-0.0455 -0.0339 -0.02 rpy=0 0 -3.14159
- joint joint3: axis 4.54273e-15 1 1.04275e-14 -> 0 1 0; origin xyz=4.08431e-07 -0.0688 0.264 rpy=-2.99502e-14 -1.6015e-14 -3.14159 -> xyz=0 -0.0688 0.264 rpy=0 0 -3.14159
- joint joint4: origin xyz=-0.0600003 -0.0688 -0.244999 rpy=2.95536e-14 8.52374e-14 -2.10585e-14 -> xyz=-0.0600003 -0.0688 -0.244999 rpy=0 0 0
- joint joint5: origin xyz=-0.0405003 0.0338995 -0.0739989 rpy=2.73264e-14 -4.32956e-16 -8.32667e-17 -> xyz=-0.0405003 0.0338995 -0.0739989 rpy=0 0 0
- joint joint6: axis 1.46014e-15 2.40808e-14 -1 -> 0 0 1; origin xyz=0.0404996 2.39858e-07 -0.0356 rpy=8.83309e-16 -5.88588e-16 7.69861e-14 -> xyz=0.0404996 0 -0.0356 rpy=3.1415926535897927 0 1.5707963267949736
- joint joint7: axis 6.86541e-15 1 0 -> 0 1 0; origin xyz=-0.0239931 0.0445119 -0.0566829 rpy=1.02229e-14 4.71845e-16 1.68314e-15 -> xyz=0.0445119 -0.0239931 0.0566829 rpy=-3.141592653589783 0 1.570796326794895
- joint joint8: axis -6.86541e-15 -1 0 -> 0 -1 0; origin xyz=0.0239931 -0.0445119 -0.0566829 rpy=9.6084e-15 -2.77556e-16 -3.77189e-15 -> xyz=-0.0445119 0.0239931 0.0566829 rpy=-3.141592653589784 0 1.5707963267949003

File: i2rt/robot_models/arm/yam_pro/v1/yam_pro.urdf (robot description, URDF)
Before this commit: robot yam_pro, 9 links, 8 joints
Joints:
- joint joint1: origin xyz=-2.49777947114e-07 0 0.0679999999995 rpy=-3.14159265359 1.57079265359 2.65359006568e-06 -> xyz=0 0 0.068 rpy=-3.14159265359 1.5708 0
- joint joint2: axis -3.58252e-15 -1 3.35753e-16 -> 0 -1 0; origin xyz=-0.0455 -0.0329 -0.02 rpy=3.36235e-16 -1.91164e-15 3.46073e-15 -> xyz=-0.0455 -0.0329 -0.02 rpy=0 0 0
- joint joint3: axis 4.54273e-15 1 1.04275e-14 -> 0 1 0; origin xyz=4.08431e-07 -0.00205 0.264 rpy=-1.07982e-14 5.71487e-14 6.40141e-16 -> xyz=0 -0.00205 0.264 rpy=0 0 0
- joint joint4: origin xyz=-0.0600003 0.0688 -0.244999 rpy=1.04275e-14 -3.65263e-14 -4.34003e-15 -> xyz=-0.0600003 0.0688 -0.244999 rpy=0 0 0
- joint joint5: origin xyz=-0.0403003 -0.0338507 -0.0739989 rpy=-8.38162e-15 -2.23269e-15 -3.35842e-15 -> xyz=-0.0403003 -0.0338507 -0.0739989 rpy=0 0 0
- joint joint6: axis 1.46014e-15 2.40808e-14 -1 -> 0 0 1; origin xyz=0.0404996 2.39858e-07 -0.0356 rpy=6.79401e-15 -1.7587e-15 8.19623e-15 -> xyz=0.0404996 0 -0.0356 rpy=3.1415926535897913 0 1.5707963267949048
- joint joint7: axis 6.86541e-15 1 0 -> 0 1 0; origin xyz=0.0239931 -0.0445119 -0.0566829 rpy=-8.79052e-15 2.82248e-16 3.14159 -> xyz=-0.0445119 0.0239931 0.0566829 rpy=3.1415926535897842 0 -1.5708
- joint joint8: axis -6.86541e-15 -1 0 -> 0 -1 0; origin xyz=-0.0239931 0.0445119 -0.0566829 rpy=-9.31451e-15 -5.70393e-16 -3.14159 -> xyz=0.0445119 -0.0239931 0.0566829 rpy=3.141592653589784 0 -1.5708

File: i2rt/robot_models/arm/yam_ultra/v1/yam_ultra.urdf (robot description, URDF)
Before this commit: robot yam_ultra, 9 links, 8 joints
Joints:
- joint joint2: axis -3.58252e-15 -1 3.2007e-16 -> 0 -1 0; origin xyz=-0.0455 0.03285 -0.02 rpy=-4.21325e-15 -1.5065e-29 9.98062e-15 -> xyz=-0.0455 0.03285 -0.02 rpy=0 0 0
- joint joint3: axis 4.54273e-15 1 1.04275e-14 -> 0 1 0; origin xyz=4.08431e-07 -0.0678 0.264 rpy=-6.20015e-15 6.98506e-29 -5.07758e-15 -> xyz=0 -0.0678 0.264 rpy=0 0 0
- joint joint4: origin xyz=-0.0600003 0.0678 -0.244999 rpy=1.04275e-14 -2.77556e-17 -4.04405e-15 -> xyz=-0.0600003 0.0678 -0.244999 rpy=0 0 0
- joint joint5: origin xyz=-0.0403003 -0.0338507 -0.0703851 rpy=-1.02186e-14 2.77556e-17 -6.12323e-17 -> xyz=-0.0403003 -0.0338507 -0.0703851 rpy=0 0 0
- joint joint6: axis 1.46014e-15 2.40808e-14 -1 -> 0 0 1; origin xyz=0.0404996 2.39858e-07 -0.0419481 rpy=7.6222e-29 -5.3963e-29 4.42535e-15 -> xyz=0.0404996 0 -0.0419481 rpy=3.141592653589793 0 1.570796326794901
- joint joint7: axis 6.86541e-15 1 0 -> 0 1 0; origin xyz=0.0239931 -0.0445119 -0.0566919 rpy=-9.48894e-15 -1.66533e-16 3.14159 -> xyz=-0.0445119 0.0239931 0.0566919 rpy=3.141592653589784 0 -1.5708
- joint joint8: axis -6.86541e-15 -1 0 -> 0 -1 0; origin xyz=-0.0239931 0.0445119 -0.0566829 rpy=-9.13119e-15 4.4964e-15 -3.14159 -> xyz=0.0445119 -0.0239931 0.0566829 rpy=3.1415926535897842 0 -1.5708

File: i2rt/robot_models/arm/yam_ultra/v2/yam_ultra.urdf (robot description, URDF)
Before this commit: robot yam_ultra, 9 links, 8 joints
Joints:
- joint joint2: axis -3.58252e-15 -1 3.2007e-16 -> 0 -1 0; origin xyz=-0.0455 0.03285 -0.02 rpy=-4.21325e-15 -1.5065e-29 9.98062e-15 -> xyz=-0.0455 0.03285 -0.02 rpy=0 0 0
- joint joint3: axis 4.54273e-15 1 1.04275e-14 -> 0 1 0; origin xyz=4.08431e-07 -0.0678 0.264 rpy=-6.20015e-15 6.98506e-29 -5.07758e-15 -> xyz=0 -0.0678 0.264 rpy=0 0 0
- joint joint4: origin xyz=-0.0600003 0.0678 -0.244999 rpy=1.04275e-14 -2.77556e-17 -4.04405e-15 -> xyz=-0.0600003 0.0678 -0.244999 rpy=0 0 0
- joint joint5: origin xyz=-0.0403003 -0.0338507 -0.0703851 rpy=-1.02186e-14 2.77556e-17 -6.12323e-17 -> xyz=-0.0403003 -0.0338507 -0.0703851 rpy=0 0 0
- joint joint6: axis 1.46014e-15 2.40808e-14 -1 -> 0 0 1; origin xyz=0.0404996 2.39858e-07 -0.0419481 rpy=7.6222e-29 -5.3963e-29 4.42535e-15 -> xyz=0.0404996 0 -0.0419481 rpy=3.141592653589793 0 1.570796326794901
- joint joint7: axis 6.86541e-15 1 0 -> 0 1 0; origin xyz=0.0239931 -0.0445119 -0.0566919 rpy=-9.48894e-15 -1.66533e-16 3.14159 -> xyz=-0.0445119 0.0239931 0.0566919 rpy=3.141592653589784 0 -1.5708
- joint joint8: axis -6.86541e-15 -1 0 -> 0 -1 0; origin xyz=-0.0239931 0.0445119 -0.0566829 rpy=-9.13119e-15 4.4964e-15 -3.14159 -> xyz=0.0445119 -0.0239931 0.0566829 rpy=3.1415926535897842 0 -1.5708

File: i2rt/robot_models/station/yam_station_crank_4310_d405/yam_station_crank_4310_d405.urdf (robot description, URDF)
Before this commit: robot yam_station_crank_4310_d405, 21 links, 20 joints
Joints:
- joint left_camera_joint: origin xyz=-0.07972864298920912 0.0016999000000607195 -0.06602077467211452 rpy=2.268922 3.673205103416066e-06 1.5707963267814042 -> xyz=0.0016999000000607195 -0.07972864298920912 0.06602077467211452 rpy=-0.8726706535897933 -3.673205103416066e-06 1.349237960600456e-11
- joint left_joint6: axis 1.46014e-15 2.40808e-14 -1 -> 2.40808e-14 1.46014e-15 1; origin xyz=0.0404996 2.39858e-07 -0.0356 rpy=8.83309e-16 -5.88588e-16 7.69861e-14 -> xyz=0.0404996 2.39858e-07 -0.0356 rpy=3.1415926535897927 -8.83309e-16 1.5707963267949736
- joint left_joint7: origin xyz=-0.0392 0.037 -0.0605 rpy=1.5708 -0 -1.5708 -> xyz=0.037 -0.0392 0.0605 rpy=-1.5707926535897934 -0 -3.14158898038469
- joint left_joint8: origin xyz=0.0392 -0.037 -0.0605 rpy=1.5708 -0 -1.5708 -> xyz=-0.037 0.0392 0.0605 rpy=-1.5707926535897934 -0 -3.14158898038469
- joint right_camera_joint: origin xyz=-0.07972864298920912 0.0016999000000607195 -0.06602077467211452 rpy=2.268922 3.673205103416066e-06 1.5707963267814042 -> xyz=0.0016999000000607195 -0.07972864298920912 0.06602077467211452 rpy=-0.8726706535897933 -3.673205103416066e-06 1.349237960600456e-11
- joint right_joint6: axis 1.46014e-15 2.40808e-14 -1 -> 2.40808e-14 1.46014e-15 1; origin xyz=0.0404996 2.39858e-07 -0.0356 rpy=8.83309e-16 -5.88588e-16 7.69861e-14 -> xyz=0.0404996 2.39858e-07 -0.0356 rpy=3.1415926535897927 -8.83309e-16 1.5707963267949736
- joint right_joint7: origin xyz=-0.0392 0.037 -0.0605 rpy=1.5708 -0 -1.5708 -> xyz=0.037 -0.0392 0.0605 rpy=-1.5707926535897934 -0 -3.14158898038469
- joint right_joint8: origin xyz=0.0392 -0.037 -0.0605 rpy=1.5708 -0 -1.5708 -> xyz=-0.037 0.0392 0.0605 rpy=-1.5707926535897934 -0 -3.14158898038469

File: i2rt/robot_models/station/yam_station_linear_4310_d405/yam_station_linear_4310_d405.urdf (robot description, URDF)
Before this commit: robot yam_station_linear_4310_d405, 21 links, 20 joints
Joints:
- joint left_camera_joint: origin xyz=-0.07043497874827391 -7.656797949839866e-08 -0.07700592901799347 rpy=2.70525 3.673205103638111e-06 1.5707963267814136 -> xyz=-7.656797949839866e-08 -0.07043497874827391 0.07700592901799347 rpy=-0.43634265358979335 -3.673205103638111e-06 1.3483053732597708e-11
- joint left_joint6: axis 1.46014e-15 2.40808e-14 -1 -> 2.40808e-14 1.46014e-15 1; origin xyz=0.0404996 2.39858e-07 -0.0356 rpy=8.83309e-16 -5.88588e-16 7.69861e-14 -> xyz=0.0404996 2.39858e-07 -0.0356 rpy=3.1415926535897927 -8.83309e-16 1.5707963267949736
- joint left_joint7: origin xyz=-0.0239931 0.0445119 -0.0566829 rpy=1.02229e-14 4.71845e-16 1.68314e-15 -> xyz=0.0445119 -0.0239931 0.0566829 rpy=-3.141592653589783 -4.71845e-16 1.570796326794895
- joint left_joint8: origin xyz=0.0239931 -0.0445119 -0.0566829 rpy=9.6084e-15 -2.77556e-16 -3.77189e-15 -> xyz=-0.0445119 0.0239931 0.0566829 rpy=-3.141592653589784 2.77556e-16 1.5707963267949003
- joint right_camera_joint: origin xyz=-0.07043497874827391 -7.656797949839866e-08 -0.07700592901799347 rpy=2.70525 3.673205103638111e-06 1.5707963267814136 -> xyz=-7.656797949839866e-08 -0.07043497874827391 0.07700592901799347 rpy=-0.43634265358979335 -3.673205103638111e-06 1.3483053732597708e-11
- joint right_joint6: axis 1.46014e-15 2.40808e-14 -1 -> 2.40808e-14 1.46014e-15 1; origin xyz=0.0404996 2.39858e-07 -0.0356 rpy=8.83309e-16 -5.88588e-16 7.69861e-14 -> xyz=0.0404996 2.39858e-07 -0.0356 rpy=3.1415926535897927 -8.83309e-16 1.5707963267949736
- joint right_joint7: origin xyz=-0.0239931 0.0445119 -0.0566829 rpy=1.02229e-14 4.71845e-16 1.68314e-15 -> xyz=0.0445119 -0.0239931 0.0566829 rpy=-3.141592653589783 -4.71845e-16 1.570796326794895
- joint right_joint8: origin xyz=0.0239931 -0.0445119 -0.0566829 rpy=9.6084e-15 -2.77556e-16 -3.77189e-15 -> xyz=-0.0445119 0.0239931 0.0566829 rpy=-3.141592653589784 2.77556e-16 1.5707963267949003

File: i2rt/robot_models/station/yambox_linear_4310_d405_decxin/yambox_linear_4310_d405_decxin.urdf (robot description, URDF)
Before this commit: robot yambox_linear_4310_d405_decxin, 21 links, 20 joints
Joints:
- joint left_camera_joint: origin xyz=-0.07043497874827391 -7.656797949839866e-08 -0.07700592901799347 rpy=2.70525 3.673205103638111e-06 1.5707963267814136 -> xyz=-7.656797949839866e-08 -0.07043497874827391 0.07700592901799347 rpy=-0.43634265358979335 -3.673205103638111e-06 1.3483053732597708e-11
- joint left_joint6: axis 1.46014e-15 2.40808e-14 -1 -> 2.40808e-14 1.46014e-15 1; origin xyz=0.0404996 2.39858e-07 -0.0356 rpy=8.83309e-16 -5.88588e-16 7.69861e-14 -> xyz=0.0404996 2.39858e-07 -0.0356 rpy=3.1415926535897927 -8.83309e-16 1.5707963267949736
- joint left_joint7: origin xyz=-0.0239931 0.0445119 -0.0566829 rpy=1.02229e-14 4.71845e-16 1.68314e-15 -> xyz=0.0445119 -0.0239931 0.0566829 rpy=-3.141592653589783 -4.71845e-16 1.570796326794895
- joint left_joint8: origin xyz=0.0239931 -0.0445119 -0.0566829 rpy=9.6084e-15 -2.77556e-16 -3.77189e-15 -> xyz=-0.0445119 0.0239931 0.0566829 rpy=-3.141592653589784 2.77556e-16 1.5707963267949003
- joint right_camera_joint: origin xyz=-0.07043497874827391 -7.656797949839866e-08 -0.07700592901799347 rpy=2.70525 3.673205103638111e-06 1.5707963267814136 -> xyz=-7.656797949839866e-08 -0.07043497874827391 0.07700592901799347 rpy=-0.43634265358979335 -3.673205103638111e-06 1.3483053732597708e-11
- joint right_joint6: axis 1.46014e-15 2.40808e-14 -1 -> 2.40808e-14 1.46014e-15 1; origin xyz=0.0404996 2.39858e-07 -0.0356 rpy=8.83309e-16 -5.88588e-16 7.69861e-14 -> xyz=0.0404996 2.39858e-07 -0.0356 rpy=3.1415926535897927 -8.83309e-16 1.5707963267949736
- joint right_joint7: origin xyz=-0.0239931 0.0445119 -0.0566829 rpy=1.02229e-14 4.71845e-16 1.68314e-15 -> xyz=0.0445119 -0.0239931 0.0566829 rpy=-3.141592653589783 -4.71845e-16 1.570796326794895
- joint right_joint8: origin xyz=0.0239931 -0.0445119 -0.0566829 rpy=9.6084e-15 -2.77556e-16 -3.77189e-15 -> xyz=-0.0445119 0.0239931 0.0566829 rpy=-3.141592653589784 2.77556e-16 1.5707963267949003
